File: ul-12/ul-12.brd (EAGLE design)
At the start: 31 x 37 mm, 39 parts, among them IC1 24C64SM, IC2 CY7C68013-56PVC, IC3 LD1117, IC4 24C64SM, IC5 24C64P, Q2 24 MHz, X1 USB-MINIB-BUV2, X2 F25D, X3 F25D

Commit message: .
Parts:
- added LED3: 3 mm bl, led:LED3MM
- added LED4: 3 mm ge, led:LED3MM
- added R16, R17: (no value), rcl:R0805
- moved R15 119.2 mm to (-30.8, -21.7), flipped to the bottom, turned to 90 degrees
- moved R14 115.2 mm to (-26.7, -21.7), flipped to the bottom, turned to 90 degrees
- moved R13 111.4 mm to (-22.5, -21.7), flipped to the bottom, turned to 90 degrees
- moved R12 107.7 mm to (-18.4, -21.7), flipped to the bottom, turned to 90 degrees
- moved R11 104.3 mm to (-14.3, -21.7), flipped to the bottom, turned to 90 degrees
- moved R10 100.5 mm to (16.0, -32.2), flipped to the bottom, turned to 270 degrees
- moved R9 98.1 mm to (-6.03, -21.7), flipped to the bottom, turned to 90 degrees
- moved R8 95.3 mm to (-1.91, -21.7), flipped to the bottom, turned to 90 degrees
- moved R7 92.9 mm to (2.22, -21.7), flipped to the bottom, turned to 90 degrees
- moved R6 88.4 mm to (13.5, -28.3), flipped to the bottom, turned to 90 degrees
- moved R1 87.9 mm to (25.9, -25.6), flipped to the bottom, turned to 90 degrees
- moved IC5 56.9 mm to (-14.9, -50.3), turned to 270 degrees
- moved R4 51.9 mm to (11.4, -67.8), flipped to the bottom, turned to 90 degrees
- moved R5 50.8 mm to (7.46, -68.3), flipped to the bottom, turned to 90 degrees
- moved IC4 45.1 mm to (-15.1, -59.1), turned to 90 degrees
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Connections:
- removed net N$45: IC4.8, IC5.8
- removed net N$47: IC4.6, IC5.6
- removed net N$48: IC4.5, IC5.5
- removed net N$51: IC4.3, IC5.3
- new net N$25: J3.13, R16.2
- new net N$26: LED3.K, R16.1
- new net N$27: J3.6, R17.2
- new net N$28: LED4.K, R17.1
- net +3V3: now also IC4.8, IC5.8, LED3.A, LED4.A
- net N$50: now also IC4.3, IC5.3
- net SCL: now also IC4.6, IC5.6
- net SDA: now also IC4.5, IC5.5
Routing:
- net +3V3: track 0.00 -> 19.9 mm
- net N$45: track 19.9 -> 0.00 mm
- net N$51: track 11.1 -> 0.00 mm
- net N$50: track 15.4 -> 26.5 mm
- net SCL: track 0.00 -> 10.5 mm
- net N$47: track 9.53 -> 0.00 mm
- net SDA: track 0.00 -> 3.08 mm
- net N$48: track 3.08 -> 0.00 mm
- net N$24: track 14.7 -> 15.9 mm

Commit message: .
Parts:
- removed X3: F25D, hs-ul:F25D
- added JP1: (no value), pinhead:1X40
- added X4: (no value), con-subd:F25HP
- added X5: F25D, hs-ul:F25D
- moved C1 102.4 mm to (71.0, 29.8)
- moved C4 102.4 mm to (77.2, 33.7)
- moved C6 102.4 mm to (83.7, 36.1)
- moved C7 102.4 mm to (67.0, 26.4)
- moved IC3 102.4 mm to (87.9, 22.5)
- moved R2 102.4 mm to (74.6, 25.6)
- moved RN1 102.4 mm to (80.0, 31.0)
- moved RN2 102.4 mm to (80.0, 40.2)
- moved RN3 102.4 mm to (80.0, 44.1)
- moved C2 102.4 mm to (66.2, 29.8)
- moved C3 102.4 mm to (86.2, 40.2)
- moved C5 102.4 mm to (68.9, 44.9)
- moved IC1 102.4 mm to (87.6, 50.4)
- moved IC2 102.4 mm to (82.1, 35.1)
- moved LED1 102.4 mm to (70.8, 47.8)
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Connections:
- net GND: now also X4.18, X4.19, X4.20, X4.21, X4.22, X4.23, X4.24, X4.25; no longer X3.18, X3.19, X3.20, X3.21, X3.22, X3.23, X3.24, X3.25
- net N$12: now also X4.2; no longer X3.2
- net N$13: now also X4.3; no longer X3.3
- net N$14: now also X4.4; no longer X3.4
- net N$15: now also X4.5; no longer X3.5
- net N$16: now also X4.6; no longer X3.6
- net N$17: now also X4.7; no longer X3.7
- net N$18: now also X4.8; no longer X3.8
- net N$19: now also X4.9; no longer X3.9
- net N$20: now also X4.10; no longer X3.10
- net N$21: now also X4.11; no longer X3.11
- net N$22: now also X4.12; no longer X3.12
- net N$23: now also X4.13; no longer X3.13
- net N$37: now also X4.17; no longer X3.17
- net N$38: now also X4.16; no longer X3.16
- net N$39: now also X4.15; no longer X3.15
- net N$40: now also X4.14; no longer X3.14
- net N$6: now also X4.1; no longer X3.1
Routing:
- net N$6: track 0.00 -> 79.1 mm
- net N$39: track 0.00 -> 75.0 mm
- net N$17: track 0.00 -> 72.2 mm, vias 0 -> 2
- net N$18: track 0.00 -> 70.8 mm, vias 0 -> 2
- net N$16: track 0.00 -> 64.8 mm, vias 0 -> 4
- net N$40: track 0.00 -> 64.1 mm, vias 0 -> 2
- net N$19: track 0.00 -> 62.1 mm, vias 0 -> 2
- net N$22: track 0.00 -> 61.4 mm
- net N$37: track 0.00 -> 59.5 mm, vias 0 -> 4
- net N$23: track 0.00 -> 57.9 mm
- net N$38: track 0.00 -> 54.3 mm, vias 0 -> 2
- net N$13: track 0.00 -> 43.3 mm
- net GND: track 222.5 -> 260.9 mm
- net N$15: track 0.00 -> 35.7 mm, vias 0 -> 2
- net N$12: track 0.00 -> 35.6 mm, vias 0 -> 2
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