File: ul-12/ul-12.sch (EAGLE design)
At the start: 39 parts, among them IC1 24C64SM, IC2 CY7C68013-56PVC, IC3 LD1117, IC4 24C64SM, IC5 24C64P, Q2 24 MHz, X1 USB-MINIB-BUV2, X2 F25D, X3 F25D

Commit message: .
Parts:
- added LED3: 3 mm bl, led:LED3MM
- added LED4: 3 mm ge, led:LED3MM
- added R16, R17: (no value), rcl:R-EU_R0805
Connections:
- removed net N$45: IC4.VCC, IC5.VCC
- removed net N$47: IC4.SCL, IC5.SCL
- removed net N$48: IC4.SDA, IC5.SDA
- removed net N$51: IC4.A2, IC5.A2
- new net N$25: J3.13, R16.2
- new net N$26: LED3.C, R16.1
- new net N$27: J3.6, R17.2
- new net N$28: LED4.C, R17.1
- net +3V3: now also IC4.VCC, IC5.VCC, LED3.A, LED4.A
- net N$50: now also IC4.A2, IC5.A2
- net SCL: now also IC4.SCL, IC5.SCL
- net SDA: now also IC4.SDA, IC5.SDA

Commit message: .
Parts:
- removed X3: F25D, hs-ul:F25D
- added JP1: (no value), pinhead:PINHD-1X40
- added X4: (no value), con-subd:F25HP
- added X5: F25D, hs-ul:F25D
Connections:
- net GND: now also X4.18, X4.19, X4.20, X4.21, X4.22, X4.23, X4.24, X4.25; no longer X3.18, X3.19, X3.20, X3.21, X3.22, X3.23, X3.24, X3.25
- net N$12: now also X4.2; no longer X3.2
- net N$13: now also X4.3; no longer X3.3
- net N$14: now also X4.4; no longer X3.4
- net N$15: now also X4.5; no longer X3.5
- net N$16: now also X4.6; no longer X3.6
- net N$17: now also X4.7; no longer X3.7
- net N$18: now also X4.8; no longer X3.8
- net N$19: now also X4.9; no longer X3.9
- net N$20: now also X4.10; no longer X3.10
- net N$21: now also X4.11; no longer X3.11
- net N$22: now also X4.12; no longer X3.12
- net N$23: now also X4.13; no longer X3.13
- net N$37: now also X4.17; no longer X3.17
- net N$38: now also X4.16; no longer X3.16
- net N$39: now also X4.15; no longer X3.15
- net N$40: now also X4.14; no longer X3.14
- net N$6: now also X4.1; no longer X3.1
