File: EAGLE_Adapter/ul-12.brd (EAGLE design)
At the start: 31 x 37 mm, 45 parts, among them IC1 24C64SM, IC2 CY7C68013-56PVC, IC3 LD1117, IC4 24C64SM, IC5 24C64P, Q2 24 MHz, X1 USB-MINIB-BUV2, X2 F25D, X5 F25D

Commit message: .
Parts:
- removed LED3: 3 mm bl, led:LED3MM
- removed LED4: 3 mm ge, led:LED3MM
- added LED5, LED6: (no value), led:SML0805
- added R18, R19: (no value), rcl:R0805
- added U$1: (no value), usb2lpt:MINI
- R16, R17: device rcl:R0805 -> rcl:0207/12
- moved R16 13.8 mm to (2.70, -50.6), turned to 0 degrees
- moved R17 7.33 mm to (-6.19, -41.1), flipped to the bottom, turned to 180 degrees
- moved X4 3.70 mm to (2.22, -88.4)
- moved R5 3.24 mm to (6.99, -64.6)
- moved R4 2.56 mm to (14.1, -63.5), turned to 270 degrees
Connections:
- net +3V3: now also LED5.A, LED6.A, R18.2, R19.2; no longer LED3.A, LED4.A
- net N$26: now also LED5.C; no longer LED3.K
- net N$28: now also LED6.C; no longer LED4.K
- net SCL: now also R19.1
- net SDA: now also R18.1
Routing:
- net N$38: track 54.3 -> 91.2 mm, vias 2 -> 0
- net N$39: track 75.0 -> 107.0 mm
- net N$18: track 70.8 -> 98.9 mm
- net N$19: track 62.1 -> 87.2 mm
- net N$37: track 59.5 -> 81.7 mm, vias 4 -> 0
- net N$49: track 0.00 -> 21.0 mm
- net N$15: track 35.7 -> 56.1 mm
- net N$17: track 72.2 -> 92.5 mm
- net N$40: track 64.1 -> 82.1 mm
- net N$16: track 64.8 -> 82.0 mm
- net +3V3: track 19.9 -> 34.6 mm
- net N$13: track 43.3 -> 57.2 mm
- net GND: track 260.9 -> 274.1 mm
- net N$6: track 79.1 -> 90.4 mm
- net N$12: track 35.6 -> 40.2 mm
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