File: EAGLE_Adapter/ul-12.sch (EAGLE design)
At the start: 45 parts, among them IC1 24C64SM, IC2 CY7C68013-56PVC, IC3 LD1117, IC4 24C64SM, IC5 24C64P, Q2 24 MHz, X1 USB-MINIB-BUV2, X2 F25D, X5 F25D

Commit message: .
Parts:
- removed LED3: 3 mm bl, led:LED3MM
- removed LED4: 3 mm ge, led:LED3MM
- added LED5, LED6: (no value), led:LEDSML0805
- added R18, R19: (no value), rcl:R-EU_R0805
- R16, R17: device rcl:R-EU_R0805 -> rcl:R-EU_0207/12
Connections:
- net +3V3: now also LED5.A, LED6.A, R18.2, R19.2; no longer LED3.A, LED4.A
- net N$26: now also LED5.C; no longer LED3.C
- net N$28: now also LED6.C; no longer LED4.C
- net SCL: now also R19.1
- net SDA: now also R18.1
